File: Hardware/pcb/PCB_main.kicad_pcb (KiCad board)
At the start: 2 copper layers, 74.2 x 80.2 mm, 46 parts, among them J1 Conn_01x02, P1 USB_C_Plug_USB2.0, SW1 BOOT OPTION, U1 exp32wroomd, U2 CH340C, U3 AMS1117-3.3

Commit message: PCB Final
Parts:
- added R16: 4.7kΩ, Resistor_SMD:R_0603_1608Metric, F.Cu at (119.1, 70.0)
- added R17: 4.7kΩ, Resistor_SMD:R_0603_1608Metric, F.Cu at (119.1, 73.8)
- moved SD1 70.6 mm to (132.6, 68.7), turned to 90 degrees
- moved C3 15.0 mm to (91.0, 112.3)
- moved C6 14.5 mm to (117.1, 82.6), turned to 0 degrees
- moved C5 13.1 mm to (117.2, 77.7), turned to 180 degrees
- moved BH1750 7.59 mm to (144.0, 81.3), turned to 0 degrees
- moved U3 7.32 mm to (90.2, 118.2), turned to 90 degrees
- moved U2 5.15 mm to (123.2, 80.1), turned to 90 degrees
- moved MQ135_D 4.93 mm to (72.5, 96.4)
- moved R10 4.93 mm to (76.4, 74.6)
- moved R11 4.93 mm to (79.6, 75.5)
- moved R13 4.93 mm to (79.7, 84.5)
- moved R14 4.93 mm to (76.3, 119.2)
- moved R15 4.93 mm to (79.9, 120.0)
- moved R4 4.93 mm to (76.2, 101.4)
- moved R5 4.93 mm to (79.6, 102.2)
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- renumbered J_DHT22 to J_DHT, LDR1 to LDR, J_MQ135_A1 to MQ135_A, J_MQ135_D1 to MQ135_D, Rain_A1 to Rain_A, Rain_D1 to Rain_D, Soil_A1 to Soil_A, Soil_D1 to Soil_D, Sound_A1 to Sound_A, Sound_D1 to Sound_D
Connections:
- C4 pad 1: Net-(D1-K) -> /5v(r)
- C5 pad 2: +5V -> +3.3V
- D1 pad 1: Net-(D1-K) -> /5v(r)
- D2 pad 1: Net-(D1-K) -> /5v(r)
- MQ135_A pad 1: +5V -> /5v(r)
- MQ135_D pad 1: +5V -> /5v(r)
- Rain_A pad 1: +5V -> /5v(r)
- Rain_D pad 1: +5V -> /5v(r)
- Sound_A pad 1: +5V -> /5v(r)
- Sound_D pad 1: +5V -> /5v(r)
- U3 pad 3: Net-(D1-K) -> /5v(r)
Routing:
- net +3.3V: track 8.94 -> 302.0 mm, vias 0 -> 12
- net /5v(r): track 0.00 -> 138.2 mm
- net SCL: track 0.00 -> 115.4 mm, vias 0 -> 12
- net SDA: track 0.00 -> 110.4 mm
- net IO39: track 0.00 -> 87.3 mm, vias 0 -> 2
- net IO33: track 0.00 -> 76.8 mm, vias 0 -> 2
- net D+: track 0.00 -> 72.9 mm, vias 0 -> 2
- net D-: track 0.00 -> 70.4 mm, vias 0 -> 2
- net IO17: track 0.00 -> 68.8 mm, vias 0 -> 2
- net IO16: track 0.00 -> 66.0 mm
- net Net-(U1A-GPIO2): track 2.81 -> 49.3 mm
- net Net-(U1A-GPIO34): track 2.80 -> 46.8 mm, vias 0 -> 2
- net Net-(U1A-GPIO32): track 2.63 -> 30.7 mm, vias 0 -> 2
- net Net-(U1A-GPIO27): track 2.60 -> 29.6 mm
- net IO18: track 0.00 -> 26.9 mm, vias 0 -> 3
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- added copper zone on B.Cu, net GND
Other:
- board size 74.2 x 80.2 mm -> 83.8 x 80.8 mm
- board text added: "ESP32 MODULAR SENSOR HUB"
